File: LabChipPCB/LabChipPCB/LabChipPCB.kicad_pcb (KiCad board)
At the start: 2 copper layers, 132.1 x 66.7 mm, 16 parts, among them J2 Raspberry_Pi_2_3_0, SW1 SW_Push, SW2 SW_Push, SW3 SW_Push, SW4 SW_Push

Commit message: pcb updates
Parts:
- moved J2 33.2 mm to (145.7, 153.3), turned to 90 degrees
- moved R3 6.51 mm to (115.3, 120.8)
- renumbered De to D2
