File: LabChipPCB/LabChipPCB/LabChipPCB.sch (KiCad schematic (older format))
At the start: 15 parts, among them J2 Raspberry_Pi_2_3_0, SW1 SW_Push, SW2 SW_Push, SW3 SW_Push, SW4 SW_Push

Commit message: Switch off power from the battery when there's power available from the Pi
Parts:
- added D?: D_Schottky, Diode_SMD:D_SOD-123, symbol Device:D_Schottky
- added Q?: FDN336P, Package_TO_SOT_SMD:SOT-23, symbol Transistor_FET:DMG2301L
- added R?: R100K, symbol Device:R_Small
- Brd1: symbol SSD1306-128x64_OLED:SSD1306 -> LabChipPCB-rescue:SSD1306-SSD1306-128x64_OLED
Connections:
- net +3V3: now also D?.1 (K), Q?.2 (S); no longer BT1.1 (+), J2.1 (3V3)
- net GND: now also R?.2
- new net: BT1.1 (+), Q?.3 (D)
- new net: D?.2 (A), J2.1 (3V3), Q?.1 (G), R?.1
Other:
- moved on the sheet: BT1, Brd1, D1, D2, D3, D4, J2, R1, R2, R3, R4, SW1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
